Commit message: various stuffs

File: description/gazebo_auto_control.xacro (robot description, xacro)
@@ -14,8 +14,8 @@
             <wheel_diameter>0.508</wheel_diameter>
             <!-- Performance tuning -->
-            <max_wheel_torque>160</max_wheel_torque>
-            <max_wheel_acceleration>3.0</max_wheel_acceleration>
+            <max_wheel_torque>200</max_wheel_torque>
+            <max_wheel_acceleration>7.0</max_wheel_acceleration>
             <!-- Optional: Wheel velocity -->
-            <max_wheel_velocity>10.0</max_wheel_velocity>
+            <!-- <max_wheel_velocity>10.0</max_wheel_velocity> -->
             <!-- Frames and TF publishing -->
             <odometry_frame>odom</odometry_frame>
@@ -25,5 +25,5 @@
             <publish_wheel_tf>true</publish_wheel_tf>
             <!-- ROS2 Compatibility Mode -->
-            <legacyMode>false</legacyMode>
+            <!-- <legacyMode>false</legacyMode> -->
         </plugin>
     </gazebo>

File: description/lidar.xacro (robot description, xacro)
@@ -22,14 +22,14 @@
         </xacro:inertial_cylinder>
     </link>
-    <!-- <gazebo reference="lidar_frame">
+    <gazebo reference="lidar_frame">
         <sensor name="laser" type="ray">
         <pose> 0 0 0 0 0 0 </pose>
-        <visualize>true</visualize>
-        <update_rate>10</update_rate>
+        <visualize>false</visualize>
+        <update_rate>50</update_rate>
         <ray>
             <scan>
                 <horizontal>
                     <samples>360</samples>
-                    <resolution>1</resolution>
+                    <!-- <resolution>1</resolution> -->
                     <min_angle>-3.14</min_angle>
                     <max_angle>3.14</max_angle>
@@ -37,12 +37,12 @@
             </scan>
             <range>
-                <min>0.3</min>
+                <min>0.2</min>
                 <max>12</max>
-                <resolution>0.01</resolution>
+                <!-- <resolution>0.01</resolution> -->
             </range>
         </ray>
         <plugin name="lidar_controller" filename="libgazebo_ros_ray_sensor.so">
             <ros>
-                <argument>-/out:=scan</argument>
+                <argument>~/out:=/scan</argument>
             </ros>
             <output_type>sensor_msgs/LaserScan</output_type>
@@ -50,4 +50,4 @@
         </plugin>
         </sensor>
-    </gazebo> -->
+    </gazebo>
 </robot>

File: description/robot.urdf.xacro (robot description, xacro)
@@ -4,5 +4,6 @@
     <xacro:include filename="gazebo_control.xacro" />
     <xacro:include filename="lidar.xacro"/>
+	<!-- <xacro:include filename="control.xacro"/> -->
     <!-- <xacro:include filename="camera.xacro"/> -->
-    <xacro:include filename="depth_camera.xacro"/>
+    <!-- <xacro:include filename="depth_camera.xacro"/> -->
 </robot>

File: description/robot_core.xacro (robot description, xacro)
@@ -19,4 +19,11 @@
     <!--BASE LINK -->
     <link name="base_link">
+    </link>
+    <joint name="base_footprint_joint" type="fixed">
+        <parent link="base_link"/>
+        <child link="base_footprint"/>
+        <origin xyz="0.0 0.0 0.0"/>
+    </joint>
+    <link name="base_footprint">
     </link>
     <!-- Chassis link -->

File: description/test.urdf.xacro (robot description, xacro)
@@ -2,14 +2,27 @@
 <robot xmlns:xacro ="http://www.ros.org/wiki/xacro"  name="robot">
     <xacro:include filename="inertial_macros.xacro"/>
-	<xacro:include filename="gazebo_auto_control.xacro"/>
-	<xacro:property name="chassis_length" value="1.778" />
-	<xacro:property name="chassis_width" value="1.27" />
-	<xacro:property name="chassis_height" value="0.05" />
+	<!-- <xacro:include filename="gazebo_auto_control.xacro"/> -->
+	<xacro:include filename="ros2_control.xacro"/>
+    <material name="orange">
+        <color rgba="1 0.3 0.1 1"/>
+    </material>
+    <material name="red">
+        <color rgba="1 0 0 1"/>
+    </material>
+	<xacro:property name="chassis_length" value="0.7" />
+	<xacro:property name="chassis_width" value="0.5" />
+	<xacro:property name="chassis_height" value="0.01" />
 	<xacro:property name="chassis_mass" value="12" />
-	<xacro:property name="wheel_radius" value="0.381" />
-	<xacro:property name="wheel_height" value="0.254" />
+	<xacro:property name="wheel_radius" value="0.15" />
+	<xacro:property name="wheel_height" value="0.10" />
 	<xacro:property name="wheel_mass" value="4" />
     <!--dummy link-->
-	<link name="base_link"/>
+	<link name="base_link"></link>
+	<joint name="joint-base_footprint" type="fixed">
+		<parent link="base_link"/>
+		<child link="base_footprint"/>
+		<origin xyz="0 0 0" rpy="0 0 0" />
+	</joint>
+	<link name="base_footprint"></link>
 	<joint name="joint-base-chassis" type="fixed">
 		<parent link="base_link"/>
@@ -24,7 +37,5 @@
 				<box size="${chassis_length} ${chassis_width} ${chassis_height}" />
 			</geometry>
-			<material name="brown">
-				<color rgba="0.3 0 0.4 1"/>
-			</material>
+			<material name="orange" />
 		</visual>
 		<collision>
@@ -34,25 +45,15 @@
 			</geometry>
 		</collision>
-		<!-- <inertial>
-			<mass value="0.4" />
-			<inertia ixx="0.00048333" iyy="0.0013367" izz="0.0018133"
-			ixy="0" ixz="0" iyz="0"/>
-		</inertial> -->
         <xacro:inertial_box mass="${chassis_mass}" x="${chassis_length}" y="${chassis_width}" z="${chassis_height}">
             <origin xyz="0 0.0 0" rpy="0 0 0"/>
         </xacro:inertial_box>
 	</link>
-	<joint name="joint-base-chassis" type="fixed">
+	<gazebo reference="chassis-link">
+        <material>Gazebo/Orange</material>
+    </gazebo>
+	<joint name="joint-chassis-upper-chassis" type="fixed">
 		<parent link="base_link"/>
-		<child link="chassis-link"/>
-		<origin xyz="0 0 ${wheel_radius}" rpy="0 0 0" />
-	</joint>
-	<gazebo reference="chassis-link">
-        <material>Gazebo/Brown</material>
-    </gazebo>
-	<joint name="joint-chassis-upper-chassis" type="fixed">
-		<parent link="chassis-link"/>
 		<child link="upper-chassis-link"/>
-		<origin xyz="0 0 1.03632" rpy="0 0 0" />
+		<origin xyz="0 0 ${0.508}" rpy="0 0 0" />
 	</joint>
 	<link name="upper-chassis-link">
@@ -62,7 +63,5 @@
 				<box size="${chassis_length} ${chassis_width} ${chassis_height}" />
 			</geometry>
-			<material name="brown">
-				<color rgba="0.3 0 0.4 1"/>
-			</material>
+			<material name="orange" />
 		</visual>
 		<collision>
@@ -82,5 +81,5 @@
 	</link>
 	<gazebo reference="upper-chassis-link">
-        <material>Gazebo/Brown</material>
+        <material>Gazebo/Orange</material>
     </gazebo>
     <material name="blue">
@@ -96,7 +95,7 @@
 	<!-- ${x_position}-${y_position}-wheel-link -->
 		<joint name="joint-chassis-${x_position}-${y_position}-stand" type="fixed">
-			<parent link="chassis-link"/>
+			<parent link="base_link"/>
 			<child link="${x_position}-${y_position}-stand-link"/>
-			<origin xyz="${x_reflect*0.3*chassis_length} ${y_reflect*(chassis_width/3+wheel_height/2)} ${(wheel_height*2)+0.04}" rpy="0 0 0" />
+			<origin xyz="${x_reflect*0.3*chassis_length} ${y_reflect*(chassis_width/3+wheel_height/2)} ${(wheel_radius*2)+0.04}" rpy="0 0 0" />
 			<axis xyz="0 0 1" />
 		</joint>
@@ -105,5 +104,5 @@
 				<origin xyz="0 0 0" rpy="0 0 0" />
 				<geometry>
-					<cylinder radius ="0.05"  length="1.03632" />
+					<cylinder radius ="0.01"  length="${0.508-0.14}" />
 				</geometry>
 				<material name="blue" />
@@ -112,5 +111,5 @@
 				<origin xyz="0 0 0" rpy="0 0 0" />
 				<geometry>
-					<cylinder radius ="0.05"  length="1.03632" />
+					<cylinder radius ="0.01"  length="${0.58-0.15}" />
 				</geometry>
 			</collision>
@@ -138,8 +137,8 @@
 	<!--LEFT SIDE-->
 	<joint name="front_left_wheel_joint" type="continuous">
-        <parent link="chassis-link"/>
+        <parent link="base_link"/>
         <child link="front_left_wheel"/>
         <axis xyz="0 0 1"/>
-        <origin xyz="${(1)*0.3*chassis_length} ${(-1)*(chassis_width/2+wheel_height/2)} 0" rpy="-${pi/2} 0 0"/>
+        <origin xyz="${(1)*0.3*chassis_length} ${(-1)*(chassis_width/2+wheel_height/2)} ${wheel_radius}" rpy="${-pi/2} 0 0"/>
     </joint>
     <link name="front_left_wheel">
@@ -160,8 +159,8 @@
     </link>
 	<joint name="rear_left_wheel_joint" type="continuous">
-        <parent link="chassis-link"/>
+        <parent link="base_link"/>
         <child link="rear_left_wheel"/>
         <axis xyz="0 0 1"/>
-        <origin xyz="${(-1)*0.3*chassis_length} ${(-1)*(chassis_width/2+wheel_height/2)} 0" rpy="-${pi/2} 0 0"/>
+        <origin xyz="${(-1)*0.3*chassis_length} ${(-1)*(chassis_width/2+wheel_height/2)} ${wheel_radius}" rpy="${-pi/2} 0 0"/>
     </joint>
     <link name="rear_left_wheel">
@@ -183,8 +182,8 @@
 	<!--RIGHT SIDE-->
 	<joint name="front_right_wheel_joint" type="continuous">
-        <parent link="chassis-link"/>
+        <parent link="base_link"/>
         <child link="front_right_wheel"/>
         <axis xyz="0 0 -1"/>
-        <origin xyz="${(1)*0.3*chassis_length} ${(1)*(chassis_width/2+wheel_height/2)} 0" rpy="${pi/2} 0 0"/>
+        <origin xyz="${(1)*0.3*chassis_length} ${(1)*(chassis_width/2+wheel_height/2)} ${wheel_radius}" rpy="${pi/2} 0 0"/>
     </joint>
     <link name="front_right_wheel">
@@ -205,8 +204,8 @@
     </link>
 	<joint name="rear_right_wheel_joint" type="continuous">
-        <parent link="chassis-link"/>
+        <parent link="base_link"/>
         <child link="rear_right_wheel"/>
         <axis xyz="0 0 -1"/>
-        <origin xyz="${(-1)*0.3*chassis_length} ${(1)*(chassis_width/2+wheel_height/2)} 0" rpy="${pi/2} 0 0"/>
+        <origin xyz="${(-1)*0.3*chassis_length} ${(1)*(chassis_width/2+wheel_height/2)} ${wheel_radius}" rpy="${pi/2} 0 0"/>
     </joint>
     <link name="rear_right_wheel">
@@ -241,12 +240,12 @@
 			<parent link="upper-chassis-link"/>
 			<child link="chassis-lidar-stand-link"/>
-			<origin xyz="0 0 ${0.4318/2}" rpy="0 0 0" />
+			<origin xyz="0 0 ${0.17/2}" rpy="0 0 0" />
 			<axis xyz="0 0 1" />
 	</joint>
 	<link name="chassis-lidar-stand-link">
 			<visual>
-				<origin xyz="0 0 0" rpy="0 0 0" />
-				<geometry>
-					<box size="0.1 0.1 0.4318" />
+				<!-- <origin xyz="0 0 0" rpy="0 0 0" /> -->
+				<geometry>
+					<box size="0.02 0.02 0.17" />
 				</geometry>
 				<material name="white" />
@@ -255,11 +254,65 @@
 				<origin xyz="0 0 0" rpy="0 0 0" />
 				<geometry>
-					<box size="0.1 0.1 0.4318" />
+					<box size="0.02 0.02 0.17" />
 				</geometry>
 			</collision>
+            <xacro:inertial_box mass="0.5" x="0.02" y="0.02" z="0.17">
+            	<origin xyz="0 0.0 0" rpy="0 0 0"/>
+        	</xacro:inertial_box>
+	</link>
+	<gazebo reference="chassis-lidar-stand-link">
+        <material>Gazebo/White</material>
+    </gazebo>
+	<!-- <joint name="joint-chassis-comm-stand" type="fixed">
+			<parent link="chassis-link"/>
+			<child link="chassis-comm-stand-link"/>
+			<origin xyz="-0.33 0 ${1.5/2}" rpy="0 ${pi/2} 0" />
+			<axis xyz="0 0 1" />
+	</joint>
+	<link name="chassis-comm-stand-link">
+			<visual>
+				<origin xyz="0 0 0" rpy="0 0 0" />
+				<geometry>
+					<box size="1.5 0.02 0.02" />
+				</geometry>
+				<material name="blue" />
+			</visual>
+			<collision>
+				<origin xyz="0 0 0" rpy="0 0 0" />
+				<geometry>
+					<box size="1.35 0.02 0.02" />
+				</geometry>
+			</collision> -->
             <!-- <xacro:inertial_cylinder mass="1" length="0.4318" radius="0.03">
                 <origin xyz="0.0 0.0 0.0" rpy="0.0 0.0 0.0"/>
             </xacro:inertial_cylinder> -->
-	</link>
+	<!-- </link>
+	<gazebo reference="chassis-comm-stand-link">
+        <material>Gazebo/Blue</material>
+    </gazebo>
+	<joint name="joint-comm_stand-sbg-mount" type="fixed">
+			<parent link="chassis-comm-stand-link"/>
+			<child link="comm_stand-sbg-mount-link"/>
+			<origin xyz="-${1.35/2} 0 0" rpy="0 0 ${pi/2}" />
+			<axis xyz="0 0 1" />
+	</joint>
+	<link name="comm_stand-sbg-mount-link">
+			<visual>
+				<origin xyz="0 0 0" rpy="0 0 0" />
+				<geometry>
+					<box size="0.8 0.02 0.02" />
+				</geometry>
+				<material name="white" />
+			</visual>
+			<collision>
+				<origin xyz="0 0 0" rpy="0 0 0" />
+				<geometry>
+					<box size="0.8 0.02 0.02" />
+				</geometry>
+			</collision> -->
+            <!-- <xacro:inertial_cylinder mass="1" length="0.4318" radius="0.03">
+                <origin xyz="0.0 0.0 0.0" rpy="0.0 0.0 0.0"/>
+            </xacro:inertial_cylinder> -->
+	<!-- </link> -->
 	<gazebo reference="chassis-lidar-stand-link">
         <material>Gazebo/White</material>
@@ -268,5 +321,5 @@
 		<parent link="chassis-lidar-stand-link"/>
 		<child link="lidar_link"/>
-		<origin xyz="0 0 ${0.4318/2}" rpy="0 0 0" />
+		<origin xyz="0 0 ${0.17/2}" rpy="0 0 0" />
 	</joint>
     <link name="lidar_link">
@@ -274,5 +327,5 @@
 			<origin xyz="0 0 0" rpy="0 0 0" />
 			<geometry>
-				<cylinder radius="0.2" length="0.10" />
+				<cylinder radius="0.05" length="0.03" />
 			</geometry>
 			<material name="black">
@@ -283,9 +336,41 @@
 			<origin xyz="0 0 0" rpy="0 0 0" />
 			<geometry>
-				<cylinder radius="0.2" length="0.10" />
+				<cylinder radius="0.05" length="0.03" />
 			</geometry>
 		</collision>
-	</link>
-	<gazebo reference="lidar-ink">
+		<xacro:inertial_cylinder mass="0.3" length="0.03" radius="0.05">
+            <origin xyz="0.0 0.0 0.0" rpy="0.0 0.0 0.0"/>
+        </xacro:inertial_cylinder>
+	</link>
+	<gazebo reference="lidar_link">
+        <sensor name="laser" type="ray">
+        <pose> 0 0 0 0 0 0 </pose>
+        <visualize>false</visualize>
+        <update_rate>50</update_rate>
+        <ray>
+            <scan>
+                <horizontal>
+                    <samples>360</samples>
+                    <!-- <resolution>1</resolution> -->
+                    <min_angle>-3.14</min_angle>
+                    <max_angle>3.14</max_angle>
+                </horizontal>
+            </scan>
+            <range>
+                <min>0.3</min>
+                <max>12</max>
+                <!-- <resolution>0.01</resolution> -->
+            </range>
+        </ray>
+        <plugin name="lidar_controller" filename="libgazebo_ros_ray_sensor.so">
+            <ros>
+                <argument>~/out:=/scan</argument>
+            </ros>
+            <output_type>sensor_msgs/LaserScan</output_type>
+            <frame_name>lidar_link</frame_name>
+        </plugin>
+        </sensor>
+    </gazebo>
+	<gazebo reference="lidar_ink">
         <material>Gazebo/Black</material>
     </gazebo>
